Commit message: Revise launch file

File: mtbc1_description/src/description/mtbc1_description.xacro (robot description, xacro)
@@ -5,4 +5,6 @@
   <xacro:property name="base_length" value="0.42"/>
   <xacro:property name="base_height" value="0.18"/>
+  <xacro:property name="c1base_len" value="0.0612"/>
+  <xacro:property name="c1base_rad" value="0.165"/>
   <xacro:property name="wheel_radius" value="0.10"/>
   <xacro:property name="wheel_width" value="0.04"/>
@@ -10,13 +12,22 @@
   <xacro:property name="wheel_zoff" value="0.05"/>
   <xacro:property name="wheel_xoff" value="0.12"/>
-  <xacro:property name="caster_xoff" value="0.14"/>
+  <xacro:property name="c1wheel_radius" value="0.0305"/>
+  <xacro:property name="c1wheel_width" value="0.00127"/>
+  <xacro:property name="c1wheel_ygap" value="0.0"/>
+  <xacro:property name="c1wheel_zoff" value="0.015"/>
+  <xacro:property name="c1wheel_xoff" value="0.00"/>
+  <!-- <xacro:property name="caster_xoff" value="0.14"/> -->
+  <xacro:property name="c1caster_xoff" value="0.123"/>
   <!-- Robot Base -->
   <link name="base_link">
     <visual>
       <geometry>
-        <box size="${base_length} ${base_width} ${base_height}"/>
+        <!--<box size="${base_length} ${base_width} ${base_height}"/> -->
+        <cylinder length="${c1base_len}" radius="${c1base_rad}"/>
       </geometry>
-      <material name="Cyan">
-        <color rgba="0 1.0 1.0 1.0"/>
+      <!--<material name="Cyan"> -->
+      <!-- <color rgba="0 1.0 1.0 1.0"/> -->
+      <material name="White">
+        <color rgba="1.0 1.0 1.0 1.0"/>
       </material>
     </visual>
@@ -27,5 +38,6 @@
     <parent link="base_link"/>
     <child link="base_footprint"/>
-    <origin xyz="0.0 0.0 ${-(wheel_radius+wheel_zoff)}" rpy="0 0 0"/>
+    <!-- <origin xyz="0.0 0.0 ${-(wheel_radius+wheel_zoff)}" rpy="0 0 0"/> -->
+    <origin xyz="0.0 0.0 ${-(c1wheel_radius+c1wheel_zoff)}" rpy="0 0 0"/>
   </joint>
   <!-- Wheels -->
@@ -35,5 +47,6 @@
         <origin xyz="0 0 0" rpy="${pi/2} 0 0"/>
         <geometry>
-            <cylinder radius="${wheel_radius}" length="${wheel_width}"/>
+            <!-- <cylinder radius="${wheel_radius}" length="${wheel_width}"/> -->
+            <cylinder radius="${c1wheel_radius}" length="${c1wheel_width}"/>
         </geometry>
         <material name="Gray">
@@ -45,5 +58,6 @@
       <parent link="base_link"/>
       <child link="${prefix}_link"/>
-      <origin xyz="${x_reflect*wheel_xoff} ${y_reflect*(base_width/2+wheel_ygap)} ${-wheel_zoff}" rpy="0 0 0"/>
+      <!-- <origin xyz="${x_reflect*wheel_xoff} ${y_reflect*(base_width/2+wheel_ygap)} ${-wheel_zoff}" rpy="0 0 0"/> -->
+      <origin xyz="${x_reflect*c1wheel_xoff} ${y_reflect*(c1base_rad+c1wheel_ygap)} ${-c1wheel_zoff}" rpy="0 0 0"/>
       <axis xyz="0 1 0"/>
     </joint>
@@ -55,8 +69,11 @@
     <visual>
       <geometry>
-        <sphere radius="${(wheel_radius+wheel_zoff-(base_height/2))}"/>
+        <!-- <sphere radius="${(wheel_radius+wheel_zoff-(base_height/2))}"/> -->
+        <sphere radius="${(c1wheel_radius+c1wheel_zoff-(c1base_len/2))}"/>
       </geometry>
-      <material name="Cyan">
-        <color rgba="0 1.0 1.0 1.0"/>
+       <!-- <material name="Cyan"> -->
+       <!-- <color rgba="0 1.0 1.0 1.0"/> -->
+        <material name="White">
+        <color rgba="1.0 1.0 1.0 1.0"/>
       </material>
     </visual>
@@ -65,5 +82,6 @@
     <parent link="base_link"/>
     <child link="front_caster"/>
-    <origin xyz="${caster_xoff} 0.0 ${-(base_height/2)}" rpy="0 0 0"/>
+    <!-- <origin xyz="${caster_xoff} 0.0 ${-(base_height/2)}" rpy="0 0 0"/> -->
+    <origin xyz="${c1caster_xoff} 0.0 ${-(c1base_len/2)}" rpy="0 0 0"/>
   </joint>
 </robot>

Commit message: Revise Wheel

File: mtbc1_description/src/description/mtbc1_description.xacro (robot description, xacro)
@@ -13,5 +13,5 @@
   <xacro:property name="wheel_xoff" value="0.12"/>
   <xacro:property name="c1wheel_radius" value="0.0305"/>
-  <xacro:property name="c1wheel_width" value="0.00127"/>
+  <xacro:property name="c1wheel_width" value="0.027"/>
   <xacro:property name="c1wheel_ygap" value="0.0"/>
   <xacro:property name="c1wheel_zoff" value="0.015"/>

Commit message: Revise Wheel Dimensiosn

File: mtbc1_description/src/description/mtbc1_description.xacro (robot description, xacro)
@@ -14,5 +14,5 @@
   <xacro:property name="c1wheel_radius" value="0.0305"/>
   <xacro:property name="c1wheel_width" value="0.027"/>
-  <xacro:property name="c1wheel_ygap" value="0.0"/>
+  <xacro:property name="c1wheel_ygap" value="0.033"/>
   <xacro:property name="c1wheel_zoff" value="0.015"/>
   <xacro:property name="c1wheel_xoff" value="0.00"/>
@@ -59,5 +59,5 @@
       <child link="${prefix}_link"/>
       <!-- <origin xyz="${x_reflect*wheel_xoff} ${y_reflect*(base_width/2+wheel_ygap)} ${-wheel_zoff}" rpy="0 0 0"/> -->
-      <origin xyz="${x_reflect*c1wheel_xoff} ${y_reflect*(c1base_rad+c1wheel_ygap)} ${-c1wheel_zoff}" rpy="0 0 0"/>
+      <origin xyz="${x_reflect*c1wheel_xoff} ${y_reflect*(c1base_rad-c1wheel_ygap)} ${-c1wheel_zoff}" rpy="0 0 0"/>
       <axis xyz="0 1 0"/>
     </joint>
