Commit message: Revise sensro_shelp xacro

File: mtbc1_description/urdf/sensors/sensors_shelf.urdf.xacro (robot description, xacro)
@@ -1,12 +1,18 @@
 <?xml version="1.0"?>
-<!-- Added to turtlebot create base and called by sensors_shelf.urdf.xacro -->
+<!-- Added to turtlebot create base and called by mtbc1_sensors.urdf.xacro -->
+<!-- Based on shell_link & joint declarion in /standard/turtlebot4_urdf.xacro -->
 <robot xmlns:xacro="http://ros.org/wiki/xacro">
-<xacro:property name="shelf_height" value="0.1225" />
+<xacro:property name="shelf_zoff" value="0.1225" />
 <xacro:property name="shelf_radius" value="0.1915" />
 <xacro:property name="shelf_length" value="0.0015" />
-<link name="base_link">
+<joint name="sensors_shelf_joint" type="fixed">
+    <parent link="base_link"/>
+    <child link="sensor_shelf_link"/>
+    <origin xyz="0 0 ${shelf_zoff}" rpy="0 0 0"/>
+<!-- Sensor Shelf Definition -->
+<link name="sensors_shelf_link">
     <visual>
         <geometry>
-            <origin xyz="0 0 ${shelf_height}" rpy="0 0 0"/>
+            <origin xyz="0 0 0" rpy="0 0 0"/>
             <cylinder radius="${shelf_radius}" length="${shelf_length}"/>
         </geometry>
@@ -20,2 +26,3 @@
 </link>
 </robot>
+8
