Commit message: Update IMU & snesors_shelf xacro

File: mtbc1_description/urdf/sensors/imu.urdf.xacro (robot description, xacro)
@@ -1,4 +1,5 @@
 <!-- From Linorobot2, mounted above Camera Bracket and called by mtbc1_sensors.urdf.xacro -->
 <robot xmlns:xacro="http://ros.org/wiki/xacro">
+  <xacro:property name="imu_zoff" value="0.141" />
   <xacro:macro name="imu">
     <link name="imu_link"/>

File: mtbc1_description/urdf/sensors/sensors_shelf.urdf.xacro (robot description, xacro)
@@ -3,5 +3,5 @@
   <!-- Based on shell_link & joint declaration in /standard/turtlebot4_urdf.xacro -->
 <robot name="Sensors" xmlns:xacro="http://ros.org/wiki/xacro">
-  <xacro:property name="shelf_zoff" value="0.1225" />
+  <xacro:property name="shelf_zoff" value="0.12485" />
   <xacro:property name="shelf_radius" value="0.075" />
   <xacro:property name="shelf_length" value="0.0015" />

Commit message: Update IMU URDF

File: mtbc1_description/urdf/sensors/imu.urdf.xacro (robot description, xacro)
@@ -1,4 +1,4 @@
 <?xml version="1.0"?>
-<!-- From Linorobot2, mounted above Camera Bracket and called by mtbc1_sensors.urdf.xacro -->
+<!-- Uses Oak-D-Lite urdf and called by mtbc1_sensors.urdf.xacro -->
 <robot xmlns:xacro="http://ros.org/wiki/xacro">
   <xacro:macro name="imu">
@@ -7,5 +7,7 @@
       <parent link="base_link"/>
       <child link="imu_link"/>
-      <origin xyz="0 0 ${imu_z_offset + shelf_zoff}" rpy="0 0 0"/>
+      <!-- <origin xyz="0 0 ${imu_z_offset + shelf_zoff}" rpy="0 0 0"/> -->
+      <origin xyz="${camera_mount_x_offset + oakd_lite_x_offset} 0 ${oakd_lite_z_offset + shelf_zoff}" rpy="0 0 0"/>
+      <!-- <origin xyz="0 0 ${imu_z_offset + shelf_zoff}" rpy="0 0 0"/> -->
     </joint>
   </xacro:macro>

File: mtbc1_description/urdf/sensors/sensors_shelf.urdf.xacro (robot description, xacro)
@@ -3,7 +3,7 @@
   <!-- Based on shell_link & joint declaration in /standard/turtlebot4_urdf.xacro -->
 <robot name="Sensors" xmlns:xacro="http://ros.org/wiki/xacro">
-  <xacro:property name="shelf_zoff" value="0.15085" />
-  <xacro:property name="shelf_radius" value="0.075" />
-  <xacro:property name="shelf_length" value="0.0015" />
+  <xacro:property name="shelf_zoff" value="${15.085*cm2m}" />
+  <xacro:property name="shelf_radius" value="${7.5*cm2m}" />
+  <xacro:property name="shelf_length" value="${.15*cm2m}" />
     <!-- Sensor Shelf Definition -->
   <link name="sensors_shelf_link">
