Commit message: Correct oakd.urdf.xacro

File: mtbc1_description/urdf/sensors/oakd.urdf.xacro (robot description, xacro)
@@ -23,5 +23,5 @@
     <visual>
       <geometry>
-        <mesh filename="package://turtlebot4_description/meshes/${name}_${model}.dae" scale="1 1 1" />
+        <mesh filename="package://mtbc1_description/meshes/${name}_${model}.dae" scale="1 1 1" />
       </geometry>
     </visual>
