Commit message: Revise colors xacro

File: mtbc1_description/urdf/create_base.urdf.xacro (robot description, xacro)
@@ -2,4 +2,16 @@
 <robot xmlns:xacro="http://ros.org/wiki/xacro">
   <xacro:property name="PI" value="3.1415926535897931" />
+  <material name="black">
+    <color rgba="0 0 0 1"/>
+  </material>
+  <material name="white">
+    <color rgba="1 1 1 1"/>
+  </material>
+  <material name="grey">
+    <color rgba="0.5 0.5 0.5 1"/>
+  </material>
+  <material name="green">
+    <color rgba="0.0 1.0 0.0 1.0"/>
+  </material>
   <xacro:macro name="create_wheel" params="prefix y_offset wheel_radius wheel_width">
     <link name="${prefix}_wheel_link">
@@ -14,4 +26,5 @@
         <cylinder radius="${wheel_radius}" length="${wheel_width}" />
       </geometry>
+      <material name="grey"/>
     </visual>
     <collision>
@@ -37,5 +50,5 @@
         <box size="0.001 0.001 0.001" />
       </geometry>
-      <material name="Green" />
+      <material name="green" />
     </visual>
     <collision>
@@ -132,5 +145,5 @@
     <xacro:create_wheel prefix="left" y_offset="${wheel_separation / 2}" wheel_radius="${wheel_radius}" wheel_width="${wheel_width}"/>
     <xacro:create_wheel prefix="right" y_offset="${wheel_separation / -2}" wheel_radius="${wheel_radius}" wheel_width="${wheel_width}"/>
-    <!--<link name="rear_wheel_link">
+    <link name="rear_wheel_link">
     <inertial>
       <origin xyz="0 0 0"/>
@@ -144,4 +157,5 @@
         <sphere radius="0.015" />
       </geometry>
+      <material name="grey"/>
     </visual>
     <collision>
@@ -157,5 +171,5 @@
       <child link="rear_wheel_link"/>
       <axis xyz="0 1 0"/>
-    </joint>-->
+    </joint>
     <link name="front_wheel_link">
     <inertial>
@@ -169,4 +183,5 @@
         <sphere radius="0.018" />
       </geometry>
+      <material name="grey"/>
     </visual>
     <collision>
@@ -184,4 +199,6 @@
       <axis xyz="0 1 0" />
     </joint>
+    <!-- Gyro Sensor -->
+    <!-- Disable Gyro Sensors
     <joint name="gyro_joint" type="fixed">
       <axis xyz="0 1 0" />
@@ -197,9 +214,12 @@
     </inertial>
     </link>
-    <!-- Simulation sensors -->
+    -->
+    <!-- Simulation Sensors -->
+    <!-- Disable Simulation
     <xacro:sim_create_base/>
     <xacro:sim_create_wall_sensor/>
     <xacro:sim_create_cliff_sensors/>
     <xacro:sim_imu/>
+     -->
   </xacro:macro>
 </robot>

File: mtbc1_description/urdf/mtbc1.urdf.xacro (robot description, xacro)
@@ -2,5 +2,5 @@
 <!-- Called by mtbc1_description.launch.py -->
 <robot name="mtbc1" xmlns:xacro="http://ros.org/wiki/xacro">
-  <xacro:include filename="$(find mtbc1_description)/urdf/common_properties.urdf.xacro" />
+<!-- <xacro:include filename="$(find mtbc1_description)/urdf/common_properties.urdf.xacro" /> -->
   <xacro:include filename="$(find mtbc1_description)/urdf/create_base.urdf.xacro" />
 <!--
