Commit message: Update sensors

File: mtbc1_description/urdf/2wdc1.urdf.xacro (robot description, xacro)
@@ -2,4 +2,5 @@
 <robot name="mtbc1" xmlns:xacro="http://ros.org/wiki/xacro">
 <!--
+<xacro:include filename="(find mtbc1_description)/urdf/common_properties.urdf.xacro" />
 <xacro:include filename="(find mtbc1_description)/urdf/mtbc1_base.urdf.xacro" />
 <xacro:include filename="(find mtbc1_description)/urdf/mtbc1_sensor.urdf.xacro" />

File: mtbc1_description/urdf/mtbc1_sensor.urdf.xacro (robot description, xacro)
@@ -3,4 +3,5 @@
   <!-- mtbc1 Sensor Models -->
   <!--<xacro:include filename="$(find irobot_create_description)/urdf/create3.urdf.xacro" /> -->
+  <xacro:include filename="$(find turtlebot4_description)/urdf/common_properties.urdf.xacro" />
   <xacro:include filename="$(find turtlebot4_description)/urdf/sensors/rplidar.urdf.xacro" />
   <xacro:include filename="$(find turtlebot4_description)/urdf/sensors/oakd.urdf.xacro" />

File: mtbc1_description/urdf/sensors/rplidar.urdf.xacro (robot description, xacro)
@@ -2,5 +2,5 @@
 <robot xmlns:xacro="http://ros.org/wiki/xacro">
 <xacro:macro name="rplidar" params="name parent_link gazebo *origin">
-  <xacro:include filename="$(find irobot_create_description)/urdf/common_properties.urdf.xacro"/>
+  <xacro:include filename="$(find mtbc1_description)/urdf/common_properties.urdf.xacro"/>
   <xacro:property name="mass"       value="0.17"/>
   <xacro:property name="length_x"   value="${7.1*cm2m}" />
@@ -18,5 +18,5 @@
     <visual>
       <geometry>
-        <mesh filename="package://turtlebot4_description/meshes/rplidar.dae" scale="1 1 1" />
+        <mesh filename="package://mtbc1_description/meshes/rplidar.dae" scale="1 1 1" />
       </geometry>
     </visual>

File: mtbc1_description/urdf/sensors/sensor_shelf.urdf.xacro (robot description, xacro)
@@ -1,3 +1,20 @@
 <?xml version="1.0"?>
 <robot xmlns:xacro="http://ros.org/wiki/xacro">
+<xacro:property name="width" value="0.0015" />
+<xacro:property name="bodylen" value="0.150" />
+<xacro:property name="height" value="0.130" />
+<link name="base_link">
+    <visual>
+        <geometry>
+            <origin xyz="0 0 ${height}" rpy="0 0 0"/>
+            <cylinder radius="${width}" length="${bodylen}"/>
+        </geometry>
+        <material name="white"/>
+    </visual>
+    <collision>
+        <geometry>
+            <cylinder radius="${width}" length="${bodylen}"/>
+        </geometry>
+    </collision>
+</link>
 </robot>

Commit message: Revise F & R Casters

File: mtbc1_description/urdf/2wdc1.urdf.xacro (robot description, xacro)
@@ -11,6 +11,6 @@
   <xacro:property name="base_length" value="0.42"/>
   <xacro:property name="base_height" value="0.18"/>
-  <xacro:property name="c1base_len" value="0.0612"/>
-  <xacro:property name="c1base_rad" value="0.165"/>
+  <xacro:property name="c1base_len" value="0.065"/>
+  <xacro:property name="c1base_rad" value="0.1915"/>
   <xacro:property name="wheel_radius" value="0.10"/>
   <xacro:property name="wheel_width" value="0.04"/>
@@ -25,4 +25,6 @@
   <!-- <xacro:property name="caster_xoff" value="0.14"/> -->
   <xacro:property name="c1caster_xoff" value="0.123"/>
+  <xacro:property name="c1fcaster_xoff" value="0.123"/>
+  <xacro:property name="c1rcaster_xoff" value="0.145"/>
   <!-- Robot Base -->
   <link name="base_link">
@@ -71,5 +73,5 @@
   <xacro:wheel prefix="drivewhl_l" x_reflect="-1" y_reflect="1" />
   <xacro:wheel prefix="drivewhl_r" x_reflect="-1" y_reflect="-1" />
-  <!-- Caster Wheel -->
+  <!-- Caster Front Wheel -->
   <link name="front_caster">
     <visual>
@@ -89,5 +91,25 @@
     <child link="front_caster"/>
     <!-- <origin xyz="${caster_xoff} 0.0 ${-(base_height/2)}" rpy="0 0 0"/> -->
-    <origin xyz="${c1caster_xoff} 0.0 ${-(c1base_len/2)}" rpy="0 0 0"/>
+    <origin xyz="${c1fcaster_xoff} 0.0 ${-(c1base_len/2)}" rpy="0 0 0"/>
+  </joint>
+  <!-- Caster Rear Wheel -->
+  <link name="Rear_caster">
+    <visual>
+      <geometry>
+        <!-- <sphere radius="${(wheel_radius+wheel_zoff-(base_height/2))}"/> -->
+        <sphere radius="${(c1wheel_radius+c1wheel_zoff-(c1base_len/2))}"/>
+      </geometry>
+       <!-- <material name="Cyan"> -->
+       <!-- <color rgba="0 1.0 1.0 1.0"/> -->
+        <material name="Black">
+        <color rgba="0.0 0.0 0.0 0.0"/>
+      </material>
+    </visual>
+  </link>
+  <joint name="caster_joint" type="fixed">
+    <parent link="base_link"/>
+    <child link="rear_caster"/>
+    <!-- <origin xyz="${caster_xoff} 0.0 ${-(base_height/2)}" rpy="0 0 0"/> -->
+    <origin xyz="${c1rcaster_xoff} 0.0 ${-(c1base_len/2)}" rpy="0 0 0"/>
   </joint>
 </robot>

Commit message: add imu xacro

File: mtbc1_description/urdf/2wdc1.urdf.xacro (robot description, xacro)
@@ -24,7 +24,9 @@
   <xacro:property name="c1wheel_xoff" value="0.00"/>
   <!-- <xacro:property name="caster_xoff" value="0.14"/> -->
-  <xacro:property name="c1caster_xoff" value="0.123"/>
+  <!-- <xacro:property name="c1caster_xoff" value="0.123"/> -->
   <xacro:property name="c1fcaster_xoff" value="0.123"/>
   <xacro:property name="c1rcaster_xoff" value="0.145"/>
+  <!--IMU Properties-->
+  <xacro:property name="imu_zoff" value="0.266"/>
   <!-- Robot Base -->
   <link name="base_link">
@@ -87,5 +89,5 @@
     </visual>
   </link>
-  <joint name="caster_joint" type="fixed">
+  <joint name="casterf_joint" type="fixed">
     <parent link="base_link"/>
     <child link="front_caster"/>
@@ -94,5 +96,5 @@
   </joint>
   <!-- Caster Rear Wheel -->
-  <link name="Rear_caster">
+  <link name="rear_caster">
     <visual>
       <geometry>
@@ -102,14 +104,14 @@
        <!-- <material name="Cyan"> -->
        <!-- <color rgba="0 1.0 1.0 1.0"/> -->
-        <material name="Black">
-        <color rgba="0.0 0.0 0.0 0.0"/>
+        <material name="White">
+        <color rgba="1.0 1.0 1.0 1.0"/>
       </material>
     </visual>
   </link>
-  <joint name="caster_joint" type="fixed">
+  <joint name="casterr_joint" type="fixed">
     <parent link="base_link"/>
     <child link="rear_caster"/>
     <!-- <origin xyz="${caster_xoff} 0.0 ${-(base_height/2)}" rpy="0 0 0"/> -->
-    <origin xyz="${c1rcaster_xoff} 0.0 ${-(c1base_len/2)}" rpy="0 0 0"/>
+    <origin xyz="${-c1rcaster_xoff} 0.0 ${-(c1base_len/2)}" rpy="0 0 0"/>
   </joint>
 </robot>

Commit message: Revise sensors xacro

File: mtbc1_description/urdf/2wdc1.urdf.xacro (robot description, xacro)
@@ -1,8 +1,9 @@
 <?xml version="1.0"?>
+<!-- Called by 2wdc1_description.launch.py -->
 <robot name="mtbc1" xmlns:xacro="http://ros.org/wiki/xacro">
 <!--
 <xacro:include filename="(find mtbc1_description)/urdf/common_properties.urdf.xacro" />
 <xacro:include filename="(find mtbc1_description)/urdf/mtbc1_base.urdf.xacro" />
-<xacro:include filename="(find mtbc1_description)/urdf/mtbc1_sensor.urdf.xacro" />
+<xacro:include filename="(find mtbc1_description)/urdf/mtbc1_sensors.urdf.xacro" />
 <xacro:include filename="(find mtbc1_description)/urdf/stacks/circlesc1.urdf.xacro />
 -->
@@ -23,6 +24,10 @@
   <xacro:property name="c1wheel_zoff" value="0.015"/>
   <xacro:property name="c1wheel_xoff" value="0.00"/>
+  <!-- Compute base_link to base_footprint_zoff from wheel radius & zoffset -->
+  <xacro:property name="base_to_footprint_zoff" value="${(c1wheel_radius+c1wheel_zoff)}"/>
   <!-- <xacro:property name="caster_xoff" value="0.14"/> -->
   <!-- <xacro:property name="c1caster_xoff" value="0.123"/> -->
+  <xacro:property name="c1fcaster_rad" value="0.00115"/>
+  <xacro:property name="c1rcaster_rad" value="0.0090"/>
   <xacro:property name="c1fcaster_xoff" value="0.123"/>
   <xacro:property name="c1rcaster_xoff" value="0.145"/>

File: mtbc1_description/urdf/common_properties.urdf.xacro (robot description, xacro)
@@ -1,4 +1,4 @@
 <?xml version="1.0" ?>
-<!-- Various useful macros -->
+<!-- Based on Turtlebot & Turtlebot4 - Various useful macros called in 2wdc1.urdf.xacro -->
 <robot name="xacro_properties" xmlns:xacro="http://ros.org/wiki/xacro">
 <!-- Conversion macros -->

File: mtbc1_description/urdf/sensors/generic_laser.urdf.xacro (robot description, xacro)
@@ -3,5 +3,5 @@
 <?xml version="1.0"?>
 <robot xmlns:xacro="http://ros.org/wiki/xacro">
-  <xacro:include filename="$(find linorobot2_description)/urdf/sensors/laser.urdf.xacro" />
+  <xacro:include filename="$(find mtbc1_description)/urdf/sensors/laser.urdf.xacro" />
   <xacro:macro name="generic_laser" params="*origin">
     <xacro:laser

File: mtbc1_description/urdf/sensors/sensors_shelf.urdf.xacro (robot description, xacro)
@@ -1,3 +1,4 @@
 <?xml version="1.0"?>
+<!-- Added to turtlebot create base and called by sensors_shelf.urdf.xacro -->
 <robot xmlns:xacro="http://ros.org/wiki/xacro">
 <xacro:property name="shelf_height" value="0.1225" />

Commit message: Revise mtbc1_sensors.urdf.xacro

File: mtbc1_description/urdf/2wdc1.urdf.xacro (robot description, xacro)
@@ -34,5 +34,5 @@
   </link>
    <!-- Robot Footprint -->
-   <link name="base_footprint"/>
+  <link name="base_footprint"/>
   <joint name="base_joint" type="fixed">
     <parent link="base_link"/>

File: mtbc1_description/urdf/mtbc1.urdf.xacro (robot description, xacro)
@@ -2,9 +2,11 @@
 <!-- Called by mtbc1_description.launch.py -->
 <robot name="mtbc1" xmlns:xacro="http://ros.org/wiki/xacro">
-<!-- <xacro:include filename="$(find mtbc1_description)/urdf/common_properties.urdf.xacro" /> -->
+  <xacro:include filename="$(find mtbc1_description)/urdf/common_properties.urdf.xacro" />
   <xacro:include filename="$(find mtbc1_description)/urdf/create_base.urdf.xacro" />
-<!--
-  <xacro:include filename="(find mtbc1_description)/urdf/mtbc1_sensors.urdf.xacro" />
-  xacro:include filename="(find mtbc1_description)/urdf/meshes/circlesc1.urdf.xacro" />
+  <!-- Test sensors_shelf.urdf.xacro -->
+  <xacro:include filename="$(find mtbc1_description)/urdf/sensors/sensors_shelf.urdf.xacro" />
+  <!--<xacro:include filename="$(find mtbc1_description)/urdf/mtbc1_sensors.urdf.xacro" /> -->
+  <!--
+  <xacro:include filename="$(find mtbc1_description)/urdf/meshes/circlesc1.urdf.xacro" />
 -->
   <xacro:create_base wheel_separation="0.26" base_diameter="0.3302">

File: mtbc1_description/urdf/mtbc1_sensors.urdf.xacro (robot description, xacro)
@@ -2,8 +2,8 @@
 <robot xmlns:xacro="http://ros.org/wiki/xacro">
   <!-- mtbc1 Sensor Models based on Turtlebot4 -->
-  <!--<xacro:include filename="$(find mtbc1_description)/urdf/sensors/oakd.urdf.xacro" /> -->
+  <!--<xacro:include filename="$(find mtbc1_description)/urdf/sensors/oakd.urdf.xacro" />
   <xacro:include filename="$(find mtbc1_description)/urdf/sensors/camera_bracket.urdf.xacro" />
   <xacro:include filename="$(find mtbc1_description)/urdf/sensors/imu.urdf.xacro" />
-  <xacro:include filename="$(find mtbc1_description)/urdf/sensors/rplidar.urdf.xacro" />
+  xacro:include filename="$(find mtbc1_description)/urdf/sensors/rplidar.urdf.xacro" /> -->
   <xacro:include filename="$(find mtbc1_description)/urdf/sensors/sensors_shelf.urdf.xacro" />
   <!-- Mechanical properties -->
@@ -29,3 +29,2 @@
   </xacro:oakd>
 </robot>
-  </robot>

File: mtbc1_description/urdf/sensors/sensors_shelf.urdf.xacro (robot description, xacro)
@@ -1,28 +1,23 @@
 <?xml version="1.0"?>
-<!-- Added to turtlebot create base and called by mtbc1_sensors.urdf.xacro -->
-<!-- Based on shell_link & joint declarion in /standard/turtlebot4_urdf.xacro -->
-<robot xmlns:xacro="http://ros.org/wiki/xacro">
-<xacro:property name="shelf_zoff" value="0.1225" />
-<xacro:property name="shelf_radius" value="0.1915" />
-<xacro:property name="shelf_length" value="0.0015" />
-<joint name="sensors_shelf_joint" type="fixed">
+  <!-- Added to mtbc1.description and called by mtbc1_sensors.urdf.xacro -->
+  <!-- Based on shell_link & joint declaration in /standard/turtlebot4_urdf.xacro -->
+<robot name="Sensors" xmlns:xacro="http://ros.org/wiki/xacro">
+  <xacro:property name="shelf_zoff" value="0.1225" />
+  <xacro:property name="shelf_radius" value="0.075" />
+  <xacro:property name="shelf_length" value="0.0015" />
+    <!-- Sensor Shelf Definition -->
+  <link name="sensors_shelf_link">
+    <visual>
+      <geometry>
+        <cylinder length="${shelf_length}" radius="${shelf_radius}"/>
+      </geometry>
+      <origin xyz="0 0 0" rpy="0 0 0"/>
+      <material name="white"/>
+    </visual>
+  </link>
+  <joint name="base_to_sensors_shelf_joint" type="fixed">
     <parent link="base_link"/>
-    <child link="sensor_shelf_link"/>
-    <origin xyz="0 0 ${shelf_zoff}" rpy="0 0 0"/>
-<!-- Sensor Shelf Definition -->
-<link name="sensors_shelf_link">
-    <visual>
-        <geometry>
-            <origin xyz="0 0 0" rpy="0 0 0"/>
-            <cylinder radius="${shelf_radius}" length="${shelf_length}"/>
-        </geometry>
-        <material name="white"/>
-    </visual>
-    <collision>
-        <geometry>
-            <cylinder radius="${shelf_radius}" length="${shelf_length}"/>
-        </geometry>
-    </collision>
-</link>
+    <child link="sensors_shelf_link"/>
+    <origin xyz="0 0 ${shelf_zoff}"/>
+  </joint>
 </robot>
-8
