Commit message: Revise 2wdc1 & mtbc1 xacro

File: mtbc1_description/urdf/mtbc1.urdf.xacro (robot description, xacro)
@@ -1,10 +1,17 @@
 <?xml version="1.0"?>
+<!-- Called by 2wdc1_description.launch.py -->
 <robot name="mtbc1" xmlns:xacro="http://ros.org/wiki/xacro">
+<!--
+<xacro:include filename="(find mtbc1_description)/urdf/common_properties.urdf.xacro" />
+<xacro:include filename="(find mtbc1_description)/urdf/mtbc1_base.urdf.xacro" />
+<xacro:include filename="(find mtbc1_description)/urdf/mtbc1_sensors.urdf.xacro" />
+xacro:include filename="(find mtbc1_description)/urdf/meshes/circlesc1.urdf.xacro" />
+-->
   <!-- Define robot constants -->
   <xacro:property name="base_width" value="0.31"/>
   <xacro:property name="base_length" value="0.42"/>
   <xacro:property name="base_height" value="0.18"/>
-  <xacro:property name="c1base_len" value="0.0612"/>
-  <xacro:property name="c1base_rad" value="0.165"/>
+  <xacro:property name="c1base_len" value="0.065"/>
+  <xacro:property name="c1base_rad" value="0.1915"/>
   <xacro:property name="wheel_radius" value="0.10"/>
   <xacro:property name="wheel_width" value="0.04"/>
@@ -17,6 +24,14 @@
   <xacro:property name="c1wheel_zoff" value="0.015"/>
   <xacro:property name="c1wheel_xoff" value="0.00"/>
+  <!-- Compute base_link to base_footprint_zoff from wheel radius & zoffset -->
+  <xacro:property name="base_to_footprint_zoff" value="${(c1wheel_radius+c1wheel_zoff)}"/>
   <!-- <xacro:property name="caster_xoff" value="0.14"/> -->
-  <xacro:property name="c1caster_xoff" value="0.123"/>
+  <!-- <xacro:property name="c1caster_xoff" value="0.123"/> -->
+  <xacro:property name="c1fcaster_rad" value="0.00115"/>
+  <xacro:property name="c1rcaster_rad" value="0.0090"/>
+  <xacro:property name="c1fcaster_xoff" value="0.123"/>
+  <xacro:property name="c1rcaster_xoff" value="0.145"/>
+  <!--IMU Properties-->
+  <xacro:property name="imu_zoff" value="0.266"/>
   <!-- Robot Base -->
   <link name="base_link">
@@ -65,5 +80,5 @@
   <xacro:wheel prefix="drivewhl_l" x_reflect="-1" y_reflect="1" />
   <xacro:wheel prefix="drivewhl_r" x_reflect="-1" y_reflect="-1" />
-  <!-- Caster Wheel -->
+  <!-- Caster Front Wheel -->
   <link name="front_caster">
     <visual>
@@ -79,9 +94,29 @@
     </visual>
   </link>
-  <joint name="caster_joint" type="fixed">
+  <joint name="casterf_joint" type="fixed">
     <parent link="base_link"/>
     <child link="front_caster"/>
     <!-- <origin xyz="${caster_xoff} 0.0 ${-(base_height/2)}" rpy="0 0 0"/> -->
-    <origin xyz="${c1caster_xoff} 0.0 ${-(c1base_len/2)}" rpy="0 0 0"/>
+    <origin xyz="${c1fcaster_xoff} 0.0 ${-(c1base_len/2)}" rpy="0 0 0"/>
+  </joint>
+  <!-- Caster Rear Wheel -->
+  <link name="rear_caster">
+    <visual>
+      <geometry>
+        <!-- <sphere radius="${(wheel_radius+wheel_zoff-(base_height/2))}"/> -->
+        <sphere radius="${(c1wheel_radius+c1wheel_zoff-(c1base_len/2))}"/>
+      </geometry>
+       <!-- <material name="Cyan"> -->
+       <!-- <color rgba="0 1.0 1.0 1.0"/> -->
+        <material name="White">
+        <color rgba="1.0 1.0 1.0 1.0"/>
+      </material>
+    </visual>
+  </link>
+  <joint name="casterr_joint" type="fixed">
+    <parent link="base_link"/>
+    <child link="rear_caster"/>
+    <!-- <origin xyz="${caster_xoff} 0.0 ${-(base_height/2)}" rpy="0 0 0"/> -->
+    <origin xyz="${-c1rcaster_xoff} 0.0 ${-(c1base_len/2)}" rpy="0 0 0"/>
   </joint>
 </robot>

Commit message: Rivised no gui-description launch

File: mtbc1_description/urdf/mtbc1.urdf.xacro (robot description, xacro)
@@ -11,28 +11,4 @@
     <mesh filename="package://mtbc1_description/meshes/create_1.dae" />
   </xacro:create_base>
-  <!-- Sensor laser (rplidar), depth (oakd) , camera_mount pose block name -->
-  <!-- xacro:name must be instantiated in the sensor device urdf.xacro -->
-  <!-- <xacro:imu/> -->
-  <!-- For linorobot2 sensor macros instanciated in mtbc1_sensors.urdf.xacro -->
-  <!--
-  <xacro:generic_laser>
-    <xacro:insert_block name="laser_pose"/>
-  </xacro:generic_laser>
-  <xacro:depth_sensor>
-    <xacro:insert_block name="depth_sensor_pose"/>
-  </xacro:depth_sensor>
-  <xacro:camera_mount>
-    <xacro:insert_block name="camera_bracket_pose"/>
-  </xacro:camera_mount>
-  <xacro:rplidar>
-    <xacro:insert_block name="rplidar_pose"/>
-  </xacro:rplidar>
-   <xacro:oakd>
-    <xacro:insert_block name="oakd_pose"/>
-  </xacro:oakd>
-  <xacro:camera_mount>
-    <xacro:insert_block name="camera_bracket_pose"/>
-  </xacro:camera_mount>
-  -->
   <!-- Do not use TB circles xacros YET
   <create/>

File: mtbc1_description/urdf/mtbc1_sensors.urdf.xacro (robot description, xacro)
@@ -25,17 +25,4 @@
   <xacro:property name="oakd_lite_y_offset"             value="${0*cm2m}"/>
   <xacro:property name="oakd_lite_z_offset"             value="${9.25385*cm2m}"/>
-  <!-- Sensor pose for laser (rplidar), depth_camera (oakd_lite), and camera_mount -->
-  <!-- From linorobot2_description 2wd_properties.urdf.xacro -->
- <!--  For linorobot2 sensor xacros , MUST match mtbc1.urdf.xacro xacro:name
-  <xacro:property name="laser_pose">
-    <origin xyz="0.12 0 0.33" rpy="0 0 0"/>
-  </xacro:property>
-  <xacro:property name="depth_sensor_pose">
-    <origin xyz="0.14 0.0 0.045" rpy="0 0 0"/>
-  </xacro:property>
-  <xacro:property name="camera_bracket_pose">
-    <origin xyz="0.14 0.0 0.045" rpy="0 0 0"/>
-  </xacro:property>
-  -->
   <!-- For Turtlebot4 sensor xacros , MUST match xacro mtbc1.urdf.xacro xacro:name-->
   <xacro:rplidar name="rplidar" parent_link="base_link">

Commit message: Functional URDF with plates & sensors

File: mtbc1_description/urdf/mtbc1.urdf.xacro (robot description, xacro)
@@ -5,12 +5,12 @@
   <xacro:include filename="$(find mtbc1_description)/urdf/create_base.urdf.xacro" />
   <!-- Test sensors_shelf.urdf.xacro -->
-  <!--<xacro:include filename="$(find mtbc1_description)/urdf/sensors/sensors_shelf.urdf.xacro" /> -->
+  <!-- <xacro:include filename="$(find mtbc1_description)/urdf/sensors/sensors_shelf.urdf.xacro" /> -->
   <xacro:include filename="$(find mtbc1_description)/urdf/mtbc1_sensors.urdf.xacro"/>
-  <!-- <xacro:include filename="$(find mtbc1_description)/urdf/stacks/circlesc1.urdf.xacro" -->
+  <xacro:include filename="$(find mtbc1_description)/urdf/stacks/circlesc1.urdf.xacro"/>
   <xacro:create_base wheel_separation="0.26" base_diameter="0.3302">
     <mesh filename="package://mtbc1_description/meshes/create_1.dae" />
   </xacro:create_base>
-  <!-- Do not use TB circles xacros YET
-  <create/>
-  <stack_circles parent="base_link"/> -->
+  <!-- TB circles xacros -->
+  <!-- <create/> -->
+  <xacro:stack_circles parent_link="base_link"/>
 </robot>

File: mtbc1_description/urdf/sensors/sensors_shelf.urdf.xacro (robot description, xacro)
@@ -3,5 +3,5 @@
   <!-- Based on shell_link & joint declaration in /standard/turtlebot4_urdf.xacro -->
 <robot name="Sensors" xmlns:xacro="http://ros.org/wiki/xacro">
-  <xacro:property name="shelf_zoff" value="0.12485" />
+  <xacro:property name="shelf_zoff" value="0.15085" />
   <xacro:property name="shelf_radius" value="0.075" />
   <xacro:property name="shelf_length" value="0.0015" />

File: mtbc1_description/urdf/stacks/circlesc1.urdf.xacro (robot description, xacro)
@@ -1,4 +1,84 @@
 <?xml version="1.0"?>
 <!-- Based on Turtlebot Create revised for Mock TurtleBot Create1 -->
-<robot name="...mtbc1" xmlns:xacro="http://ros.org/wiki/xacro">
+<robot name="mtbc1_hardware" xmlns:xacro="http://ros.org/wiki/xacro">
+  <xacro:macro name="stack_circles" params="parent_link">
+    <joint name="plate_0_joint" type="fixed">
+      <origin xyz="-0.04334 0  0.06775704" rpy="0 0 0" />
+      <parent link="${parent_link}"/>
+      <child link="plate_0_link" />
+    </joint>
+    <link name="plate_0_link">
+      <inertial>
+        <mass value="0.01" />
+        <origin xyz="0 0 0" />
+        <inertia ixx="0.01" ixy="0.0" ixz="0.0"
+          iyy="0.01" iyz="0.0"
+          izz="0.01" />
+      </inertial>
+      <visual>
+        <origin xyz=" 0 0 0 " rpy="0 0 0" />
+        <geometry>
+          <mesh filename="package://mtbc1_description/meshes/stacks/circles/plate_0_logo.dae"/>
+        </geometry>
+      </visual>
+      <collision>
+        <origin xyz="0.0 0.0 0.0" rpy="0 0 0" />
+        <geometry>
+          <box size="0.233502 0.314845 0.006401"/>
+        </geometry>
+      </collision>
+    </link>
+    <joint name="plate_1_joint" type="fixed">
+      <origin xyz="0.04068 0 0.05715" rpy="0 0 0" />
+      <parent link="plate_0_link"/>
+      <child link="plate_1_link" />
+    </joint>
+    <link name="plate_1_link">
+      <inertial>
+        <mass value="0.1" />
+        <origin xyz="0 0 0" />
+        <inertia ixx="0.01" ixy="0.0" ixz="0.0"
+          iyy="0.01" iyz="0.0"
+          izz="0.01" />
+      </inertial>
+      <visual>
+        <origin xyz=" 0 0 0 " rpy="0 0 0" />
+        <geometry>
+          <mesh filename="package://mtbc1_description/meshes/stacks/circles/plate_1_logo.dae"/>
+        </geometry>
+      </visual>
+      <collision>
+        <origin xyz="0.0 0.0 0.0" rpy="0 0 0" />
+        <geometry>
+          <box size="0.314856 0.314856 0.006401"/>
+        </geometry>
+      </collision>
+    </link>
+    <joint name="plate_3_joint" type="fixed">
+      <origin xyz="-0.01316 0 0.2063496" rpy="0 0 0" />
+      <parent link="plate_1_link"/>
+      <child link="plate_3_link" />
+    </joint>
+    <link name="plate_3_link">
+      <inertial>
+        <mass value="0.01" />
+        <origin xyz="0 0 0" />
+        <inertia ixx="0.0001" ixy="0.0" ixz="0.0"
+          iyy="0.0001" iyz="0.0"
+          izz="0.0001" />
+      </inertial>
+      <visual>
+        <origin xyz=" 0 0 0 " rpy="0 0 0" />
+        <geometry>
+          <mesh filename="package://mtbc1_description/meshes/stacks/circles/plate_2_logo.dae"/>
+        </geometry>
+      </visual>
+      <collision>
+        <origin xyz="0.0 0.0 0.0" rpy="0 0 0" />
+        <geometry>
+          <box size="0.288 0.315 0.006401"/>
+        </geometry>
+      </collision>
+    </link>
+  </xacro:macro>
 </robot>
