Commit message: Update color xacro

File: mtbc1_description/urdf/common_properties.urdf.xacro (robot description, xacro)
@@ -7,8 +7,39 @@
   <xacro:property name="in2m"    value="0.0254"/>
   <xacro:property name="deg2rad" value="${pi/180.0}"/>
-  <!-- Material colors -->
+<!-- Material colors -->
+<!-- From Turtlebot -->
+    <xacro:property name="material_white">
+    <material name="white">
+      <color rgba="1 1 1 1"/>
+    </material>
+  </xacro:property>
   <xacro:property name="material_black">
     <material name="black">
       <color rgba="0.1 0.1 0.1 1"/>
+    </material>
+  </xacro:property>
+  <xacro:property name="material_grey">
+    <material name="grey">
+      <color rgba="0.5 0.5 0.5 1"/>
+    </material>
+  </xacro:property>
+  <xacro:property name="material_light_grey">
+    <material name="light_grey">
+      <color rgba="0.6 0.6 0.6 1"/>
+    </material>
+  </xacro:property>
+  <xacro:property name="material_dark_grey">
+    <material name="dark_grey">
+      <color rgba="0.3 0.3 0.3 1"/>
+    </material>
+  </xacro:property>
+  <xacro:property name="material_black">
+    <material name="black">
+      <color rgba="0.1 0.1 0.1 1"/>
+    </material>
+  </xacro:property>
+  <xacro:property name="material_red">
+    <material name="red">
+      <color rgba="1 0 0 1"/>
     </material>
   </xacro:property>

Commit message: Update xacro

File: mtbc1_description/urdf/common_properties.urdf.xacro (robot description, xacro)
@@ -63,3 +63,2 @@
     </visual>
   </xacro:macro>
-</robot>

File: mtbc1_description/urdf/mtbc1_base.urdf.xacro (robot description, xacro)
@@ -85,3 +85,3 @@
     <origin xyz="${c1caster_xoff} 0.0 ${-(c1base_len/2)}" rpy="0 0 0"/>
   </joint>
-<.robot>
+</robot>

File: mtbc1_description/urdf/mtbc1_sensor.urdf.xacro (robot description, xacro)
@@ -1,5 +1,5 @@
 <?xml version="1.0" ?>
 <robot xmlns:xacro="http://ros.org/wiki/xacro">
-  <!-- mtbc1 Sensor Models -->
+  <!-- mtbc1 Sensor Models based on Turtlebot4 -->
   <!--<xacro:include filename="$(find irobot_create_description)/urdf/create3.urdf.xacro" /> -->
   <xacro:include filename="$(find turtlebot4_description)/urdf/common_properties.urdf.xacro" />
@@ -17,14 +17,3 @@
   <xacro:property name="oakd_lite_y_offset"             value="${0*cm2m}"/>
   <xacro:property name="oakd_lite_z_offset"             value="${9.25385*cm2m}"/>
-  <!-- Turtlebot4 sensor definitions -->
-  <xacro:rplidar name="rplidar" parent_link="base_link" gazebo="$(arg gazebo)">
-    <origin xyz="${rplidar_x_offset} ${rplidar_y_offset} ${rplidar_z_offset + base_link_z_offset}"
-            rpy="0 0 ${pi/2}"/>
-  </xacro:rplidar>
-  <xacro:camera_bracket name="oakd_camera_bracket" parent_link="base_link">
-    <origin xyz="${camera_mount_x_offset} ${camera_mount_y_offset} ${camera_mount_z_offset + base_link_z_offset}"/>
-  </xacro:camera_bracket>
-  <xacro:oakd model="lite" parent_link="oakd_camera_bracket">
-    <origin xyz="${oakd_lite_x_offset} ${oakd_lite_y_offset} ${oakd_lite_z_offset}"/>
-  </xacro:oakd>
-</robot>
+  </robot>

File: mtbc1_description/urdf/sensors/sensor_shelf.urdf.xacro (robot description, xacro)
@@ -1,12 +1,12 @@
 <?xml version="1.0"?>
 <robot xmlns:xacro="http://ros.org/wiki/xacro">
-<xacro:property name="width" value="0.0015" />
-<xacro:property name="bodylen" value="0.150" />
-<xacro:property name="height" value="0.130" />
+<xacro:property name="shelf_height" value="0.1225" />
+<xacro:property name="shelf_radius" value="0.1915" />
+<xacro:property name="shelf_length" value="0.0015" />
 <link name="base_link">
     <visual>
         <geometry>
-            <origin xyz="0 0 ${height}" rpy="0 0 0"/>
-            <cylinder radius="${width}" length="${bodylen}"/>
+            <origin xyz="0 0 ${shelf_height}" rpy="0 0 0"/>
+            <cylinder radius="${shelf_radius}" length="${shelf_length}"/>
         </geometry>
         <material name="white"/>
@@ -14,5 +14,5 @@
     <collision>
         <geometry>
-            <cylinder radius="${width}" length="${bodylen}"/>
+            <cylinder radius="${shelf_radius}" length="${shelf_length}"/>
         </geometry>
     </collision>

Commit message: Corrected create_base.urdf.xacro

File: mtbc1_description/urdf/common_properties.urdf.xacro (robot description, xacro)
@@ -63,2 +63,3 @@
     </visual>
   </xacro:macro>
+</robot>

File: mtbc1_description/urdf/mtbc1.urdf.xacro (robot description, xacro)
@@ -1,122 +1,13 @@
 <?xml version="1.0"?>
-<!-- Called by 2wdc1_description.launch.py -->
+<!-- Called by mtbc1_description.launch.py -->
 <robot name="mtbc1" xmlns:xacro="http://ros.org/wiki/xacro">
+  <xacro:include filename="$(find mtbc1_description)/urdf/common_properties.urdf.xacro" />
+  <xacro:include filename="$(find mtbc1_description)/urdf/create_base.urdf.xacro" />
 <!--
-<xacro:include filename="(find mtbc1_description)/urdf/common_properties.urdf.xacro" />
-<xacro:include filename="(find mtbc1_description)/urdf/mtbc1_base.urdf.xacro" />
-<xacro:include filename="(find mtbc1_description)/urdf/mtbc1_sensors.urdf.xacro" />
-xacro:include filename="(find mtbc1_description)/urdf/meshes/circlesc1.urdf.xacro" />
+  <xacro:include filename="(find mtbc1_description)/urdf/mtbc1_sensors.urdf.xacro" />
+  xacro:include filename="(find mtbc1_description)/urdf/meshes/circlesc1.urdf.xacro" />
 -->
-  <!-- Define robot constants -->
-  <xacro:property name="base_width" value="0.31"/>
-  <xacro:property name="base_length" value="0.42"/>
-  <xacro:property name="base_height" value="0.18"/>
-  <xacro:property name="c1base_len" value="0.065"/>
-  <xacro:property name="c1base_rad" value="0.1915"/>
-  <xacro:property name="wheel_radius" value="0.10"/>
-  <xacro:property name="wheel_width" value="0.04"/>
-  <xacro:property name="wheel_ygap" value="0.025"/>
-  <xacro:property name="wheel_zoff" value="0.05"/>
-  <xacro:property name="wheel_xoff" value="0.12"/>
-  <xacro:property name="c1wheel_radius" value="0.0305"/>
-  <xacro:property name="c1wheel_width" value="0.027"/>
-  <xacro:property name="c1wheel_ygap" value="0.033"/>
-  <xacro:property name="c1wheel_zoff" value="0.015"/>
-  <xacro:property name="c1wheel_xoff" value="0.00"/>
-  <!-- Compute base_link to base_footprint_zoff from wheel radius & zoffset -->
-  <xacro:property name="base_to_footprint_zoff" value="${(c1wheel_radius+c1wheel_zoff)}"/>
-  <!-- <xacro:property name="caster_xoff" value="0.14"/> -->
-  <!-- <xacro:property name="c1caster_xoff" value="0.123"/> -->
-  <xacro:property name="c1fcaster_rad" value="0.00115"/>
-  <xacro:property name="c1rcaster_rad" value="0.0090"/>
-  <xacro:property name="c1fcaster_xoff" value="0.123"/>
-  <xacro:property name="c1rcaster_xoff" value="0.145"/>
-  <!--IMU Properties-->
-  <xacro:property name="imu_zoff" value="0.266"/>
-  <!-- Robot Base -->
-  <link name="base_link">
-    <visual>
-      <geometry>
-        <!--<box size="${base_length} ${base_width} ${base_height}"/> -->
-        <cylinder length="${c1base_len}" radius="${c1base_rad}"/>
-      </geometry>
-      <!--<material name="Cyan"> -->
-      <!-- <color rgba="0 1.0 1.0 1.0"/> -->
-      <material name="White">
-        <color rgba="1.0 1.0 1.0 1.0"/>
-      </material>
-    </visual>
-  </link>
-   <!-- Robot Footprint -->
-   <link name="base_footprint"/>
-  <joint name="base_joint" type="fixed">
-    <parent link="base_link"/>
-    <child link="base_footprint"/>
-    <!-- <origin xyz="0.0 0.0 ${-(wheel_radius+wheel_zoff)}" rpy="0 0 0"/> -->
-    <origin xyz="0.0 0.0 ${-(c1wheel_radius+c1wheel_zoff)}" rpy="0 0 0"/>
-  </joint>
-  <!-- Wheels -->
-  <xacro:macro name="wheel" params="prefix x_reflect y_reflect">
-    <link name="${prefix}_link">
-      <visual>
-        <origin xyz="0 0 0" rpy="${pi/2} 0 0"/>
-        <geometry>
-            <!-- <cylinder radius="${wheel_radius}" length="${wheel_width}"/> -->
-            <cylinder radius="${c1wheel_radius}" length="${c1wheel_width}"/>
-        </geometry>
-        <material name="Gray">
-          <color rgba="0.5 0.5 0.5 1.0"/>
-        </material>
-      </visual>
-    </link>
-    <joint name="${prefix}_joint" type="continuous">
-      <parent link="base_link"/>
-      <child link="${prefix}_link"/>
-      <!-- <origin xyz="${x_reflect*wheel_xoff} ${y_reflect*(base_width/2+wheel_ygap)} ${-wheel_zoff}" rpy="0 0 0"/> -->
-      <origin xyz="${x_reflect*c1wheel_xoff} ${y_reflect*(c1base_rad-c1wheel_ygap)} ${-c1wheel_zoff}" rpy="0 0 0"/>
-      <axis xyz="0 1 0"/>
-    </joint>
-  </xacro:macro>
-  <xacro:wheel prefix="drivewhl_l" x_reflect="-1" y_reflect="1" />
-  <xacro:wheel prefix="drivewhl_r" x_reflect="-1" y_reflect="-1" />
-  <!-- Caster Front Wheel -->
-  <link name="front_caster">
-    <visual>
-      <geometry>
-        <!-- <sphere radius="${(wheel_radius+wheel_zoff-(base_height/2))}"/> -->
-        <sphere radius="${(c1wheel_radius+c1wheel_zoff-(c1base_len/2))}"/>
-      </geometry>
-       <!-- <material name="Cyan"> -->
-       <!-- <color rgba="0 1.0 1.0 1.0"/> -->
-        <material name="White">
-        <color rgba="1.0 1.0 1.0 1.0"/>
-      </material>
-    </visual>
-  </link>
-  <joint name="casterf_joint" type="fixed">
-    <parent link="base_link"/>
-    <child link="front_caster"/>
-    <!-- <origin xyz="${caster_xoff} 0.0 ${-(base_height/2)}" rpy="0 0 0"/> -->
-    <origin xyz="${c1fcaster_xoff} 0.0 ${-(c1base_len/2)}" rpy="0 0 0"/>
-  </joint>
-  <!-- Caster Rear Wheel -->
-  <link name="rear_caster">
-    <visual>
-      <geometry>
-        <!-- <sphere radius="${(wheel_radius+wheel_zoff-(base_height/2))}"/> -->
-        <sphere radius="${(c1wheel_radius+c1wheel_zoff-(c1base_len/2))}"/>
-      </geometry>
-       <!-- <material name="Cyan"> -->
-       <!-- <color rgba="0 1.0 1.0 1.0"/> -->
-        <material name="White">
-        <color rgba="1.0 1.0 1.0 1.0"/>
-      </material>
-    </visual>
-  </link>
-  <joint name="casterr_joint" type="fixed">
-    <parent link="base_link"/>
-    <child link="rear_caster"/>
-    <!-- <origin xyz="${caster_xoff} 0.0 ${-(base_height/2)}" rpy="0 0 0"/> -->
-    <origin xyz="${-c1rcaster_xoff} 0.0 ${-(c1base_len/2)}" rpy="0 0 0"/>
-  </joint>
+  <xacro:create_base wheel_separation="0.26" base_diameter="0.3302">
+    <mesh filename="package://mtbc1_description/meshes/create_1.dae" />
+  </xacro:create_base>
 </robot>

Commit message: Revise to TB4 Varients

File: mtbc1_description/urdf/common_properties.urdf.xacro (robot description, xacro)
@@ -2,4 +2,43 @@
 <!-- Based on Turtlebot & Turtlebot4 - Various useful macros called in mtbc1.urdf.xacro -->
 <robot name="xacro_properties" xmlns:xacro="http://ros.org/wiki/xacro">
+  <xacro:macro name="inertial_cuboid_with_pose" params="mass x y z *origin">
+    <inertial>
+      <mass value="${mass}" />
+      <xacro:insert_block name="origin"/>
+      <inertia ixx="${(1/12) * mass * (y*y + z*z)}" ixy="0.0" ixz="0.0"
+        iyy="${(1/12) * mass * (x*x + z*z)}" iyz="0.0"
+        izz="${(1/12) * mass * (x*x + y*y)}" />
+    </inertial>
+  </xacro:macro>
+  <xacro:macro name="inertial_cuboid" params="mass x y z">
+    <xacro:inertial_cuboid_with_pose mass="${mass}" x="${x}" y="${y}" z="${z}">
+      <origin xyz="0 0 0" />
+    </xacro:inertial_cuboid_with_pose>
+  </xacro:macro>
+  <xacro:macro name="inertial_cylinder_with_pose" params="mass radius length *origin">
+    <inertial>
+      <xacro:insert_block name="origin"/>
+      <mass value="${mass}" />
+      <inertia ixx="${(1/12) * mass * (3*radius*radius + length*length)}" ixy="0.0" ixz="0.0"
+        iyy="${(1/12) * mass * (3*radius*radius + length*length)}" iyz="0.0"
+        izz="${(1/2) * mass * (radius*radius)}" />
+    </inertial>
+  </xacro:macro>
+  <xacro:macro name="inertial_cylinder" params="mass radius length">
+    <xacro:inertial_cylinder_with_pose mass="${mass}" radius="${radius}" length="${length}">
+      <origin xyz="0 0 0" />
+    </xacro:inertial_cylinder_with_pose>
+  </xacro:macro>
+  <xacro:macro name="inertial_sphere" params="mass radius">
+    <inertial>
+      <mass value="${mass}" />
+      <inertia ixx="${(2/5) * mass * radius * radius}" ixy="0.0" ixz="0.0"
+	             iyy="${(2/5) * mass * radius * radius}" iyz="0.0"
+	             izz="${(2/5) * mass * radius * radius}" />
+    </inertial>
+  </xacro:macro>
+  <xacro:macro name="inertial_dummy">
+    <xacro:inertial_cuboid mass="0.01" x="0.01" y="0.01" z="0.01"/>
+  </xacro:macro>
 <!-- Conversion macros -->
   <xacro:property name="cm2m"    value="${1/100.0}"/>

File: mtbc1_description/urdf/mtbc1.urdf.xacro (robot description, xacro)
@@ -5,11 +5,36 @@
   <xacro:include filename="$(find mtbc1_description)/urdf/create_base.urdf.xacro" />
   <!-- Test sensors_shelf.urdf.xacro -->
-  <xacro:include filename="$(find mtbc1_description)/urdf/sensors/sensors_shelf.urdf.xacro" />
-    <!--<xacro:include filename="$(find mtbc1_description)/urdf/mtbc1_sensors.urdf.xacro" /> -->
-  <xacro:include filename="$(find mtbc1_description)/urdf/stacks/circlesc1.urdf.xacro" />
+  <!--<xacro:include filename="$(find mtbc1_description)/urdf/sensors/sensors_shelf.urdf.xacro" /> -->
+  <xacro:include filename="$(find mtbc1_description)/urdf/mtbc1_sensors.urdf.xacro"/>
+  <!-- <xacro:include filename="$(find mtbc1_description)/urdf/stacks/circlesc1.urdf.xacro" -->
   <xacro:create_base wheel_separation="0.26" base_diameter="0.3302">
     <mesh filename="package://mtbc1_description/meshes/create_1.dae" />
   </xacro:create_base>
+  <!-- Sensor laser (rplidar), depth (oakd) , camera_mount pose block name -->
+  <!-- xacro:name must be instantiated in the sensor device urdf.xacro -->
+  <!-- <xacro:imu/> -->
+  <!-- For linorobot2 sensor macros instanciated in mtbc1_sensors.urdf.xacro -->
+  <!--
+  <xacro:generic_laser>
+    <xacro:insert_block name="laser_pose"/>
+  </xacro:generic_laser>
+  <xacro:depth_sensor>
+    <xacro:insert_block name="depth_sensor_pose"/>
+  </xacro:depth_sensor>
+  <xacro:camera_mount>
+    <xacro:insert_block name="camera_bracket_pose"/>
+  </xacro:camera_mount>
+  <xacro:rplidar>
+    <xacro:insert_block name="rplidar_pose"/>
+  </xacro:rplidar>
+   <xacro:oakd>
+    <xacro:insert_block name="oakd_pose"/>
+  </xacro:oakd>
+  <xacro:camera_mount>
+    <xacro:insert_block name="camera_bracket_pose"/>
+  </xacro:camera_mount>
+  -->
+  <!-- Do not use TB circles xacros YET
   <create/>
-  <stack_circles parent="base_link/>"/>
+  <stack_circles parent="base_link"/> -->
 </robot>

File: mtbc1_description/urdf/mtbc1_sensors.urdf.xacro (robot description, xacro)
@@ -2,28 +2,49 @@
 <robot xmlns:xacro="http://ros.org/wiki/xacro">
   <!-- mtbc1 Sensor Models based on Turtlebot4 -->
-  <!--<xacro:include filename="$(find mtbc1_description)/urdf/sensors/oakd.urdf.xacro" />
+  <!--
+  <xacro:include filename="$(find mtbc1_description)/urdf/sensors/imu.urdf.xacro" />  -->
+  <xacro:include filename="$(find mtbc1_description)/urdf/sensors/oakd.urdf.xacro" />
   <xacro:include filename="$(find mtbc1_description)/urdf/sensors/camera_bracket.urdf.xacro" />
+  <xacro:include filename="$(find mtbc1_description)/urdf/sensors/rplidar.urdf.xacro" />
+  <!-- linorobot2 sensor names -->
+  <!--
   <xacro:include filename="$(find mtbc1_description)/urdf/sensors/imu.urdf.xacro" />
-  <xacro:include filename="$(find mtbc1_description)/urdf/sensors/rplidar.urdf.xacro" />   -->
+  <xacro:include filename="$(find mtbc1_description)/urdf/sensors/generic_laser.urdf.xacro" />
+  <xacro:include filename="$(find mtbc1_description)/urdf/sensors/depth_sensor.urdf.xacro" />
+  -->
   <xacro:include filename="$(find mtbc1_description)/urdf/sensors/sensors_shelf.urdf.xacro" />
+  <!-- TB4 sensors definitions from turtlebot4.urdf.xacro,revised for turtlebot createC1 with gazebo parameters deleted-->
   <!-- Mechanical properties -->
-  <xacro:property name="rplidar_x_offset"              value="${0.393584*cm2m}"/>
+  <xacro:property name="rplidar_x_offset"              value="${0*cm2m}"/>
   <xacro:property name="rplidar_y_offset"              value="${0*cm2m}"/>
-  <xacro:property name="rplidar_z_offset"              value="${7.529272*cm2m}"/>
+  <xacro:property name="rplidar_z_offset"              value="${4.7*cm2m}"/>
   <xacro:property name="camera_mount_x_offset"         value="${-9*cm2m}"/>
   <xacro:property name="camera_mount_y_offset"         value="${0*cm2m}"/>
-  <xacro:property name="camera_mount_z_offset"         value="${2.914772*cm2m}"/>
+  <xacro:property name="camera_mount_z_offset"         value="${0*cm2m}"/>
   <xacro:property name="oakd_lite_x_offset"             value="${5.294026*cm2m}"/>
   <xacro:property name="oakd_lite_y_offset"             value="${0*cm2m}"/>
   <xacro:property name="oakd_lite_z_offset"             value="${9.25385*cm2m}"/>
-  <!-- MtbC1 sensor definitions with gazebo parameters deleted-->
+  <!-- Sensor pose for laser (rplidar), depth_camera (oakd_lite), and camera_mount -->
+  <!-- From linorobot2_description 2wd_properties.urdf.xacro -->
+ <!--  For linorobot2 sensor xacros , MUST match mtbc1.urdf.xacro xacro:name
+  <xacro:property name="laser_pose">
+    <origin xyz="0.12 0 0.33" rpy="0 0 0"/>
+  </xacro:property>
+  <xacro:property name="depth_sensor_pose">
+    <origin xyz="0.14 0.0 0.045" rpy="0 0 0"/>
+  </xacro:property>
+  <xacro:property name="camera_bracket_pose">
+    <origin xyz="0.14 0.0 0.045" rpy="0 0 0"/>
+  </xacro:property>
+  -->
+  <!-- For Turtlebot4 sensor xacros , MUST match xacro mtbc1.urdf.xacro xacro:name-->
   <xacro:rplidar name="rplidar" parent_link="base_link">
-    <origin xyz="${rplidar_x_offset} ${rplidar_y_offset} ${rplidar_z_offset + base_link_z_offset}"
-            rpy="0 0 ${pi/2}"/>
+    <origin xyz="${rplidar_x_offset} ${rplidar_y_offset} ${rplidar_z_offset + shelf_zoff}"
+            rpy="0 0 0"/>
   </xacro:rplidar>
   <xacro:camera_bracket name="oakd_camera_bracket" parent_link="base_link">
-    <origin xyz="${camera_mount_x_offset} ${camera_mount_y_offset} ${camera_mount_z_offset + base_link_z_offset}"/>
+    <origin xyz="${camera_mount_x_offset} ${camera_mount_y_offset} ${camera_mount_z_offset + shelf_zoff}"/>
   </xacro:camera_bracket>
-  <xacro:oakd model="lite" parent_link="oakd_camera_bracket">
+  <xacro:oakd name="oakd" model="lite" parent_link="oakd_camera_bracket">
     <origin xyz="${oakd_lite_x_offset} ${oakd_lite_y_offset} ${oakd_lite_z_offset}"/>
   </xacro:oakd>

Commit message: Revise imu link

File: mtbc1_description/urdf/common_properties.urdf.xacro (robot description, xacro)
@@ -83,4 +83,9 @@
     </material>
   </xacro:property>
+  <xacro:property name="material_dark_blue">
+    <material name="dark_blue">
+      <color rgba="0 0 255 1"/>
+    </material>
+  </xacro:property>
   <!-- Material macros -->
   <xacro:macro name="material_black">

File: mtbc1_description/urdf/sensors/imu.urdf.xacro (robot description, xacro)
@@ -1,13 +1,12 @@
+<?xml version="1.0"?>
 <!-- From Linorobot2, mounted above Camera Bracket and called by mtbc1_sensors.urdf.xacro -->
 <robot xmlns:xacro="http://ros.org/wiki/xacro">
-  <xacro:property name="imu_zoff" value="0.141" />
   <xacro:macro name="imu">
     <link name="imu_link"/>
-    <joint name="imu_to_base_link" type="fixed">
+    <joint name="imu_to_base_joint" type="fixed">
       <parent link="base_link"/>
       <child link="imu_link"/>
-      <!-- <origin xyz="0 0 0" rpy="0 0 0"/> -->
-      <origin xyz="0 0 ${imu_zoff}" rpy="0 0 0"/>
+      <origin xyz="0 0 ${imu_z_offset + shelf_zoff}" rpy="0 0 0"/>
     </joint>
- </xacro:macro>
+  </xacro:macro>
 </robot>
