Commit message: Update Meshes & xacros

File: mtbc1_description/urdf/mtbc1_sensors.urdf.xacro (robot description, xacro)
@@ -4,5 +4,4 @@
   <!--<xacro:include filename="$(find irobot_create_description)/urdf/create3.urdf.xacro" /> -->
   <xacro:include filename="$(find turtlebot4_description)/urdf/common_properties.urdf.xacro" />
-  <xacro:include filename="$(find turtlebot4_description)/urdf/sensors/generic_laser.urdf.xacro" />
   <!--<xacro:include filename="$(find turtlebot4_description)/urdf/sensors/oakd.urdf.xacro" /> -->
   <xacro:include filename="$(find turtlebot4_description)/urdf/sensors/camera_bracket.urdf.xacro" />
@@ -17,3 +16,15 @@
   <xacro:property name="oakd_lite_y_offset"             value="${0*cm2m}"/>
   <xacro:property name="oakd_lite_z_offset"             value="${9.25385*cm2m}"/>
+  <!-- MtbC1 sensor definitions with gazebo parameters deleted-->
+  <xacro:rplidar name="rplidar" parent_link="base_link">
+    <origin xyz="${rplidar_x_offset} ${rplidar_y_offset} ${rplidar_z_offset + base_link_z_offset}"
+            rpy="0 0 ${pi/2}"/>
+  </xacro:rplidar>
+  <xacro:camera_bracket name="oakd_camera_bracket" parent_link="base_link">
+    <origin xyz="${camera_mount_x_offset} ${camera_mount_y_offset} ${camera_mount_z_offset + base_link_z_offset}"/>
+  </xacro:camera_bracket>
+  <xacro:oakd model="lite" parent_link="oakd_camera_bracket">
+    <origin xyz="${oakd_lite_x_offset} ${oakd_lite_y_offset} ${oakd_lite_z_offset}"/>
+  </xacro:oakd>
+</robot>
   </robot>

File: mtbc1_description/urdf/sensors/imu.urdf.xacro (robot description, xacro)
@@ -1,3 +1,3 @@
-<!-- From Linorobot2, mounted above Camera Bracket -->
+<!-- From Linorobot2, mounted above Camera Bracket and called by mtbc1_sensors.urdf.xacro -->
 <robot xmlns:xacro="http://ros.org/wiki/xacro">
   <xacro:macro name="imu">

File: mtbc1_description/urdf/sensors/mtbc1_sensors.urdf.xacro (robot description, xacro)
@@ -3,7 +3,7 @@
 <robot xmlns:xacro="http://ros.org/wiki/xacro">
 <xacro:include filename="(find mtbc1_description)/urdf/sensors_shelf.urdf.xacro"/>
-<xacro:include filename="(find mtbc1_description)/urdf/rplidar.urdf.xacro"/>
-<xacro:include filename="(find mtbc1_description)/urdf/camera_bracket.urdf.xacro"/>
-<xacro:include filename="(find mtbc1_description)/urdf/imu.urdf.xacro"/>
+<xacro:include filename="(find mtbc1_description)/urdf/sensors/rplidar.urdf.xacro"/>
+<xacro:include filename="(find mtbc1_description)/urdf/sensors/camera_bracket.urdf.xacro"/>
+<xacro:include filename="(find mtbc1_description)/urdf/sensors/imu.urdf.xacro"/>
 <!-- Mechanical properties -->
   <xacro:property name="rplidar_x_offset"              value="${0.393584*cm2m}"/>
@@ -16,5 +16,5 @@
   <xacro:property name="oakd_lite_y_offset"             value="${0*cm2m}"/>
   <xacro:property name="oakd_lite_z_offset"             value="${9.25385*cm2m}"/>
-  <!-- Turtlebot4 sensor definitions with gazebo parameters deleted-->
+  <!-- MtbC1 sensor definitions with gazebo parameters deleted-->
   <xacro:rplidar name="rplidar" parent_link="base_link">
     <origin xyz="${rplidar_x_offset} ${rplidar_y_offset} ${rplidar_z_offset + base_link_z_offset}"

File: mtbc1_description/urdf/stacks/circlesc1.urdf.xacro (robot description, xacro)
@@ -1,3 +1,4 @@
 <?xml version="1.0"?>
+<!-- Based on Turtlebot Create revised for Mock TurtleBot Create1 -->
 <robot name="turtlebot_hardware" xmlns:xacro="http://ros.org/wiki/xacro">
 <xacro:macro name="turtlebot_spacer" params="parent number x_loc y_loc z_loc">
@@ -18,5 +19,5 @@
         <origin xyz=" 0 0 0 " rpy="0 0 0" />
         <geometry>
-          <mesh filename="package://turtlebot_description/meshes/stacks/circles/68-02403-125_Spacer.dae"/>
+          <mesh filename="package://mtbc1_description/meshes/stacks/circles/68-02403-125_Spacer.dae"/>
         </geometry>
       </visual>
@@ -46,5 +47,5 @@
         <origin xyz=" 0 0 0 " rpy="0 0 0" />
         <geometry>
-          <mesh filename="package://turtlebot_description/meshes/stacks/circles/68-04552-2000-RA_Turtlebot_M-F_Standoff.dae"/>
+          <mesh filename="package://mtbc1_description/meshes/stacks/circles/68-04552-2000-RA_Turtlebot_M-F_Standoff.dae"/>
         </geometry>
       </visual>
@@ -74,5 +75,5 @@
         <origin xyz=" 0 0 0 " rpy="0 0 0" />
         <geometry>
-          <mesh filename="package://turtlebot_description/meshes/stacks/circles/68-02421-8000-RA_Turtlebot_F-F_Standoff.dae"/>
+          <mesh filename="package://mtbc1_description/meshes/stacks/circles/68-02421-8000-RA_Turtlebot_F-F_Standoff.dae"/>
         </geometry>
       </visual>
@@ -106,5 +107,5 @@
         <origin xyz=" 0 0 0 " rpy="0 0 0" />
         <geometry>
-          <mesh filename="package://turtlebot_description/meshes/stacks/circles/plate_0_logo.dae"/>
+          <mesh filename="package://mtbc1_description/meshes/stacks/circles/plate_0_logo.dae"/>
         </geometry>
       </visual>
@@ -168,5 +169,5 @@
         <origin xyz=" 0 0 0 " rpy="0 0 0" />
         <geometry>
-          <mesh filename="package://turtlebot_description/meshes/stacks/circles/plate_1_logo.dae"/>
+          <mesh filename="package://mtbc1_description/meshes/stacks/circles/plate_1_logo.dae"/>
         </geometry>
       </visual>
@@ -194,5 +195,5 @@
         <origin xyz=" 0 0 0 " rpy="0 0 0" />
         <geometry>
-          <mesh filename="package://turtlebot_description/meshes/stacks/circles/plate_2_logo.dae"/>
+          <mesh filename="package://mtbc1_description/meshes/stacks/circles/plate_2_logo.dae"/>
         </geometry>
       </visual>

Commit message: Revise imu link

File: mtbc1_description/urdf/mtbc1_sensors.urdf.xacro (robot description, xacro)
@@ -2,6 +2,5 @@
 <robot xmlns:xacro="http://ros.org/wiki/xacro">
   <!-- mtbc1 Sensor Models based on Turtlebot4 -->
-  <!--
-  <xacro:include filename="$(find mtbc1_description)/urdf/sensors/imu.urdf.xacro" />  -->
+  <xacro:include filename="$(find mtbc1_description)/urdf/sensors/imu.urdf.xacro" />
   <xacro:include filename="$(find mtbc1_description)/urdf/sensors/oakd.urdf.xacro" />
   <xacro:include filename="$(find mtbc1_description)/urdf/sensors/camera_bracket.urdf.xacro" />
@@ -25,4 +24,8 @@
   <xacro:property name="oakd_lite_y_offset"             value="${0*cm2m}"/>
   <xacro:property name="oakd_lite_z_offset"             value="${9.25385*cm2m}"/>
+  <xacro:property name="imu_z_offset" value="${14.1*cm2m}" />
+  <xacro:property name="imu_length" value="${2.55*cm2m}" />
+  <xacro:property name="imu_width" value="${1.55*cm2m}" />
+  <xacro:property name="imu_height" value="${0.16*cm2m}" />
   <!-- For Turtlebot4 sensor xacros , MUST match xacro mtbc1.urdf.xacro xacro:name-->
   <xacro:rplidar name="rplidar" parent_link="base_link">
@@ -36,3 +39,4 @@
     <origin xyz="${oakd_lite_x_offset} ${oakd_lite_y_offset} ${oakd_lite_z_offset}"/>
   </xacro:oakd>
+  <xacro:imu/>
 </robot>

Commit message: Update IMU URDF

File: mtbc1_description/urdf/mtbc1_sensors.urdf.xacro (robot description, xacro)
@@ -6,10 +6,4 @@
   <xacro:include filename="$(find mtbc1_description)/urdf/sensors/camera_bracket.urdf.xacro" />
   <xacro:include filename="$(find mtbc1_description)/urdf/sensors/rplidar.urdf.xacro" />
-  <!-- linorobot2 sensor names -->
-  <!--
-  <xacro:include filename="$(find mtbc1_description)/urdf/sensors/imu.urdf.xacro" />
-  <xacro:include filename="$(find mtbc1_description)/urdf/sensors/generic_laser.urdf.xacro" />
-  <xacro:include filename="$(find mtbc1_description)/urdf/sensors/depth_sensor.urdf.xacro" />
-  -->
   <xacro:include filename="$(find mtbc1_description)/urdf/sensors/sensors_shelf.urdf.xacro" />
   <!-- TB4 sensors definitions from turtlebot4.urdf.xacro,revised for turtlebot createC1 with gazebo parameters deleted-->
@@ -25,7 +19,4 @@
   <xacro:property name="oakd_lite_z_offset"             value="${9.25385*cm2m}"/>
   <xacro:property name="imu_z_offset" value="${14.1*cm2m}" />
-  <xacro:property name="imu_length" value="${2.55*cm2m}" />
-  <xacro:property name="imu_width" value="${1.55*cm2m}" />
-  <xacro:property name="imu_height" value="${0.16*cm2m}" />
   <!-- For Turtlebot4 sensor xacros , MUST match xacro mtbc1.urdf.xacro xacro:name-->
   <xacro:rplidar name="rplidar" parent_link="base_link">

File: mtbc1_description/urdf/sensors/imu.urdf.xacro (robot description, xacro)
@@ -7,7 +7,5 @@
       <parent link="base_link"/>
       <child link="imu_link"/>
-      <!-- <origin xyz="0 0 ${imu_z_offset + shelf_zoff}" rpy="0 0 0"/> -->
       <origin xyz="${camera_mount_x_offset + oakd_lite_x_offset} 0 ${oakd_lite_z_offset + shelf_zoff}" rpy="0 0 0"/>
-      <!-- <origin xyz="0 0 ${imu_z_offset + shelf_zoff}" rpy="0 0 0"/> -->
     </joint>
   </xacro:macro>
